File: pcb/snowman_pcb.kicad_pcb (KiCad board)
At the start: 2 copper layers, 51.9 x 95.2 mm, 11 parts, among them SW1 SW_SPDT

Commit message: Pcb - all components in place
Parts:
- removed the G*** at (67.0, 78.6) (x4)
- added G*** (x3): LOGO, LOGO, F.Cu at (67.0, 78.6)
- added REF**: MountingHole_2.2mm_M2, MountingHole:MountingHole_2.2mm_M2, F.Cu at (60.7, 36.6)
- D5: footprint snowman_pcb:LED_1206_3216Metric_ReverseMount_NoHole1.8x2.4mm -> snowman_pcb:LED_D3.0mm_Horizontal_O1.27mm_Z2.0mm; moved to F.Cu
- moved D5 19.0 mm to (86.9, 75.4), turned to 0 degrees
- moved D4 18.6 mm to (68.1, 79.0), turned to 180 degrees
- moved D3 1.58 mm to (66.8, 58.2)
- turned D2 to 0 degrees
Connections:
- SW1 pad 1: Net-(SW1-Pad1) -> (no net)
Routing:
- net Net-(D1-Pad2): track 0.00 -> 80.8 mm
- net +3V0: track 0.00 -> 41.5 mm
- net GND: track 0.00 -> 12.6 mm, vias 0 -> 4
- added copper zone on B.Cu, net GND
- added copper zone on F.Cu, net GND

Commit message: Signature
Parts:
- removed the G*** at (67.0, 78.6) (x3)
- added G*** (x3): LOGO, LOGO, F.Cu at (67.0, 78.6)
- added Ref**: Val**, snowman_pcb:signature, B.Cu at (59.4, 76.5)

Commit message: Finished revision 1
Parts:
- removed the G*** at (67.0, 78.6) (x2)
- added G*** (x2): LOGO, LOGO, F.Cu at (67.0, 78.6)
Routing:
- net +3V0: track 41.5 -> 39.3 mm
Changed lines of the file:
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@@
     (visible_elements FFFFFF7F)
     (pcbplotparams
-      (layerselection 0x010f0_80000001)
+      (layerselection 0x010f0_ffffffff)
       (usegerberextensions false)
       (usegerberattributes false)
@@
       (linewidth 0.100000)
       (plotframeref false)
-      (viasonmask false)
+      (viasonmask true)
       (mode 1)
       (useauxorigin false)
@@
       (outputformat 1)
       (mirror false)
-      (drillshape 1)
+      (drillshape 0)
       (scaleselection 1)
       (outputdirectory "gerbers/"))
@@
     (add_net GND)
     (add_net "Net-(D1-Pad2)")
+    (add_net "Net-(SW1-Pad1)")
   )
   (module snowman_pcb:signature (layer B.Cu)
@@
   (via (at 69.67 100.05) (size 0.6) (drill 0.4) (layers F.Cu B.Cu) (net 1))
   (via (at 69.342 116.586) (size 0.6) (drill 0.4) (layers F.Cu B.Cu) (net 1))
-  (segment (start 58.632123 95.76) (end 57.922123 96.47) (width 0.25) (layer B.Cu) (net 2))
-  (segment (start 69.23 95.76) (end 58.632123 95.76) (width 0.25) (layer B.Cu) (net 2))
   (segment (start 57.387935 96.47) (end 57.123416 96.205481) (width 0.25) (layer B.Cu) (net 2))
   (segment (start 57.922123 96.47) (end 57.387935 96.47) (width 0.25) (layer B.Cu) (net 2))
@@
   (segment (start 64.904999 116.834999) (end 64.904999 100.085001) (width 0.25) (layer B.Cu) (net 2))
   (segment (start 69.23 121.16) (end 64.904999 116.834999) (width 0.25) (layer B.Cu) (net 2))
+  (segment (start 61.002936 100.085001) (end 57.123416 96.205481) (width 0.25) (layer B.Cu) (net 2))
+  (segment (start 64.904999 100.085001) (end 61.002936 100.085001) (width 0.25) (layer B.Cu) (net 2))
   (segment (start 66.68 86.099859) (end 66.68 78.97) (width 0.25) (layer B.Cu) (net 3))
   (segment (start 57.873416 94.906443) (end 66.68 86.099859) (width 0.25) (layer B.Cu) (net 3))
@@
     (connect_pads (clearance 0.508))
     (min_thickness 0.254)
-    (keepout (tracks not_allowed) (vias not_allowed) (copperpour allowed))
+    (keepout (tracks not_allowed) (vias not_allowed) (copperpour not_allowed))
     (fill (arc_segments 32) (thermal_gap 0.508) (thermal_bridge_width 0.508))
     (polygon
       (pts
-        (xy 69.24 80.06) (xy 69.07 77.77) (xy 67.28 77.68) (xy 67.056 80.01)
+        (xy 69.342 80.06) (xy 69.342 77.77) (xy 67.056 77.724) (xy 67.056 80.01)
       )
     )
@@
     (connect_pads (clearance 0.508))
     (min_thickness 0.254)
-    (keepout (tracks not_allowed) (vias not_allowed) (copperpour allowed))
+    (keepout (tracks not_allowed) (vias not_allowed) (copperpour not_allowed))
     (fill (arc_segments 32) (thermal_gap 0.508) (thermal_bridge_width 0.508))
     (polygon
       (pts
-        (xy 65.54 57.28) (xy 67.96 57.06) (xy 67.88 59.27) (xy 65.67 59.27)
+        (xy 65.54 57.15) (xy 67.818 57.15) (xy 67.818 59.182) (xy 65.532 59.182)
       )
     )
@@
     (connect_pads (clearance 0.508))
     (min_thickness 0.254)
-    (keepout (tracks not_allowed) (vias not_allowed) (copperpour allowed))
+    (keepout (tracks not_allowed) (vias not_allowed) (copperpour not_allowed))
     (fill (arc_segments 32) (thermal_gap 0.508) (thermal_bridge_width 0.508))
     (polygon
       (pts
-        (xy 66.3 48.6) (xy 68.51 48.69) (xy 68.39 50.68) (xy 66.39 50.6)
+        (xy 66.294 48.514) (xy 68.326 48.514) (xy 68.326 50.8) (xy 66.294 50.8)
       )
     )
@@
     (connect_pads (clearance 0.508))
     (min_thickness 0.254)
-    (keepout (tracks not_allowed) (vias not_allowed) (copperpour allowed))
+    (keepout (tracks not_allowed) (vias not_allowed) (copperpour not_allowed))
     (fill (arc_segments 32) (thermal_gap 0.508) (thermal_bridge_width 0.508))
     (polygon
       (pts
-        (xy 59.93 50.05) (xy 62.01 50.22) (xy 61.71 52.26) (xy 59.97 52.21)
+        (xy 59.93 50.038) (xy 61.976 50.038) (xy 61.976 52.324) (xy 59.944 52.324)
       )
     )

Commit message: Remove invalid footprint, add readme and licence
Parts:
- removed the G*** at (67.0, 78.6) (x2)
- added G*** (x2): LOGO, LOGO, F.Cu at (67.0, 78.6)
- BT1: footprint snowman_pcb:BatteryHolder_THT_CR2032 -> Battery:BatteryHolder_Keystone_3009_1x2450
Changed lines of the file:
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@@
     (add_net "Net-(SW1-Pad1)")
+  )
+  (module Battery:BatteryHolder_Keystone_3009_1x2450 (layer B.Cu)
+    (at 69.23 108.46 270)
+    (descr http://www.keyelco.com/product-pdf.cfm?p=787)
+    (tags "Keystone type 3009 coin cell retainer")
+    (fp_text reference BT1 (at 0 14.4 90) (layer B.SilkS)
+      (effects (font (size 1 1) (thickness 0.15)) (justify mirror))
+    )
+    (fp_text value Battery_Cell (at 0 -14 90) (layer B.Fab)
+      (effects (font (size 1 1) (thickness 0.15)) (justify mirror))
+    )
+    (fp_line (start -4.45 12.55) (end -13.35 6.7) (layer B.CrtYd) (width 0.05))
+    (fp_line (start -3.8 12.9) (end 3.8 12.9) (layer B.Fab) (width 0.1))
+    (fp_line (start 3.8 12.9) (end 3.8 12.2) (layer B.Fab) (width 0.1))
+    (fp_line (start -3.8 12.9) (end -3.8 12.2) (layer B.Fab) (width 0.1))
+    (fp_line (start -3.8 12.2) (end -12.7 6.35) (layer B.Fab) (width 0.1))
+    (fp_line (start 3.8 12.2) (end 12.7 6.35) (layer B.Fab) (width 0.1))
+    (fp_line (start -3.95 12.25) (end -12.85 6.4) (layer B.SilkS) (width 0.12))
+    (fp_line (start -3.95 13.05) (end -3.95 12.25) (layer B.SilkS) (width 0.12))
+    (fp_line (start -3.95 13.05) (end 3.95 13.05) (layer B.SilkS) (width 0.12))
+    (fp_line (start 3.95 13.05) (end 3.95 12.25) (layer B.SilkS) (width 0.12))
+    (fp_line (start 3.95 12.25) (end 12.85 6.4) (layer B.SilkS) (width 0.12))
+    (fp_line (start 4.45 12.55) (end 13.35 6.7) (layer B.CrtYd) (width 0.05))
+    (fp_line (start -4.45 13.55) (end -4.45 12.55) (layer B.CrtYd) (width 0.05))
+    (fp_line (start -4.45 13.55) (end 4.45 13.55) (layer B.CrtYd) (width 0.05))
+    (fp_line (start 4.45 13.55) (end 4.45 12.55) (layer B.CrtYd) (width 0.05))
+    (fp_line (start -12.7 6.35) (end -12.7 -7.3) (layer B.Fab) (width 0.1))
+    (fp_line (start 12.7 6.35) (end 12.7 -7.3) (layer B.Fab) (width 0.1))
+    (fp_line (start 13.35 -1.95) (end 13.35 -7.3) (layer B.CrtYd) (width 0.05))
+    (fp_line (start -13.35 6.7) (end -13.35 1.95) (layer B.CrtYd) (width 0.05))
+    (fp_line (start -13.35 -1.95) (end -13.35 -7.3) (layer B.CrtYd) (width 0.05))
+    (fp_line (start 13.35 6.7) (end 13.35 1.95) (layer B.CrtYd) (width 0.05))
+    (fp_line (start -12.85 6.4) (end -12.85 1.9) (layer B.SilkS) (width 0.12))
+    (fp_line (start 12.85 6.4) (end 12.85 1.9) (layer B.SilkS) (width 0.12))
+    (fp_circle (center 0 0) (end 12.25 0) (layer Dwgs.User) (width 0.15))
+    (fp_arc (start -10.15 -7.25) (end -10.15 -9.8) (angle -90) (layer B.Fab) (width 0.1))
+    (fp_arc (start 10.15 -7.25) (end 10.15 -9.8) (angle 90) (layer B.Fab) (width 0.1))
+    (fp_line (start -12.85 -1.9) (end -12.85 -7.3) (layer B.SilkS) (width 0.12))
+    (fp_line (start 12.85 -1.9) (end 12.85 -7.3) (layer B.SilkS) (width 0.12))
+    (fp_arc (start 10.15 -7.25) (end 10.15 -9.95) (angle 90) (layer B.SilkS) (width 0.12))
+    (fp_arc (start -10.15 -7.25) (end -10.15 -9.95) (angle -90) (layer B.SilkS) (width 0.12))
+    (fp_arc (start 0 -21) (end -9.6 -9.58) (angle -80) (layer B.Fab) (width 0.1))
+    (fp_arc (start -10.15 -9) (end -10.15 -9.8) (angle 45) (layer B.Fab) (width 0.1))
+    (fp_arc (start 10.15 -9) (end 10.15 -9.8) (angle -45) (layer B.Fab) (width 0.1))
+    (fp_arc (start -10.15 -9) (end -10.15 -9.95) (angle 45) (layer B.SilkS) (width 0.12))
+    (fp_arc (start 10.15 -9) (end 10.15 -9.95) (angle -45) (layer B.SilkS) (width 0.12))
+    (fp_arc (start 0 -21) (end -9.55 -9.73) (angle -80) (layer B.SilkS) (width 0.12))
+    (fp_arc (start -12.7 0) (end -13.35 -1.95) (angle -143) (layer B.CrtYd) (width 0.05))
+    (fp_arc (start 12.7 0) (end 13.35 -1.95) (angle 143) (layer B.CrtYd) (width 0.05))
+    (fp_arc (start -10.15 -7.25) (end -10.15 -10.45) (angle -90) (layer B.CrtYd) (width 0.05))
+    (fp_arc (start 10.15 -7.25) (end 10.15 -10.45) (angle 90) (layer B.CrtYd) (width 0.05))
+    (fp_arc (start -10.15 -9) (end -10.15 -10.45) (angle 45) (layer B.CrtYd) (width 0.05))
+    (fp_arc (start 10.15 -9) (end 10.15 -10.45) (angle -45) (layer B.CrtYd) (width 0.05))
+    (fp_arc (start 0 -21) (end -9.15 -10.05) (angle -3.2) (layer B.CrtYd) (width 0.05))
+    (fp_arc (start 0 0) (end 0 -12.8) (angle -41.7) (layer B.CrtYd) (width 0.05))
+    (fp_arc (start 0 -21) (end 9.15 -10.05) (angle 3.2) (layer B.CrtYd) (width 0.05))
+    (fp_arc (start 0 0) (end 0 -12.8) (angle 41.7) (layer B.CrtYd) (width 0.05))
+    (fp_text user %R (at 0 0 90) (layer B.Fab)
+      (effects (font (size 1 1) (thickness 0.15)) (justify mirror))
+    )
+    (pad 2 smd rect (at 0 0 270) (size 8 8) (layers B.Cu B.Mask)
+      (net 1 GND))
+    (pad 1 thru_hole circle (at 12.7 0 270) (size 3 3) (drill 1.9) (layers *.Cu *.Mask)
+      (net 2 +3V0))
+    (pad 1 thru_hole circle (at -12.7 0 270) (size 3 3) (drill 1.9) (layers *.Cu *.Mask)
+      (net 2 +3V0))
+    (model ${KISYS3DMOD}/Battery.3dshapes/BatteryHolder_Keystone_3009_1x2450.wrl
+      (at (xyz 0 0 0))
+      (scale (xyz 1 1 1))
+      (rotate (xyz 0 0 0))
+    )
   )
   (module snowman_pcb:signature (layer B.Cu)
@@
       (at (xyz 0 0 0))
       (scale (xyz 1 1 1))
-      (rotate (xyz 0 0 0))
-    )
-  )
-  (module snowman_pcb:BatteryHolder_THT_CR2032 (layer B.Cu)
-    (at 69.23 108.46 270)
-    (descr http://www.keyelco.com/product-pdf.cfm?p=787)
-    (tags "Keystone type 3009 coin cell retainer")
-    (fp_text reference BT1 (at 0 14.4 90) (layer B.SilkS)
-      (effects (font (size 1 1) (thickness 0.15)) (justify mirror))
-    )
-    (fp_text value Battery_Cell (at 0 -14 90) (layer B.Fab)
-      (effects (font (size 1 1) (thickness 0.15)) (justify mirror))
-    )
-    (fp_line (start -4.45 12.55) (end -13.35 6.7) (layer B.CrtYd) (width 0.05))
-    (fp_line (start -3.8 12.9) (end 3.8 12.9) (layer B.Fab) (width 0.1))
-    (fp_line (start 3.8 12.9) (end 3.8 12.2) (layer B.Fab) (width 0.1))
-    (fp_line (start -3.8 12.9) (end -3.8 12.2) (layer B.Fab) (width 0.1))
-    (fp_line (start -3.8 12.2) (end -12.7 6.35) (layer B.Fab) (width 0.1))
-    (fp_line (start 3.8 12.2) (end 12.7 6.35) (layer B.Fab) (width 0.1))
-    (fp_line (start -3.95 12.25) (end -12.85 6.4) (layer B.SilkS) (width 0.12))
-    (fp_line (start -3.95 13.05) (end -3.95 12.25) (layer B.SilkS) (width 0.12))
-    (fp_line (start -3.95 13.05) (end 3.95 13.05) (layer B.SilkS) (width 0.12))
-    (fp_line (start 3.95 13.05) (end 3.95 12.25) (layer B.SilkS) (width 0.12))
-    (fp_line (start 3.95 12.25) (end 12.85 6.4) (layer B.SilkS) (width 0.12))
-    (fp_line (start 4.45 12.55) (end 13.35 6.7) (layer B.CrtYd) (width 0.05))
-    (fp_line (start -4.45 13.55) (end -4.45 12.55) (layer B.CrtYd) (width 0.05))
-    (fp_line (start -4.45 13.55) (end 4.45 13.55) (layer B.CrtYd) (width 0.05))
-    (fp_line (start 4.45 13.55) (end 4.45 12.55) (layer B.CrtYd) (width 0.05))
-    (fp_line (start -12.7 6.35) (end -12.7 -7.3) (layer B.Fab) (width 0.1))
-    (fp_line (start 12.7 6.35) (end 12.7 -7.3) (layer B.Fab) (width 0.1))
-    (fp_line (start 13.35 -1.95) (end 13.35 -7.3) (layer B.CrtYd) (width 0.05))
-    (fp_line (start -13.35 6.7) (end -13.35 1.95) (layer B.CrtYd) (width 0.05))
-    (fp_line (start -13.35 -1.95) (end -13.35 -7.3) (layer B.CrtYd) (width 0.05))
-    (fp_line (start 13.35 6.7) (end 13.35 1.95) (layer B.CrtYd) (width 0.05))
-    (fp_line (start -12.85 6.4) (end -12.85 1.9) (layer B.SilkS) (width 0.12))
-    (fp_line (start 12.85 6.4) (end 12.85 1.9) (layer B.SilkS) (width 0.12))
-    (fp_circle (center 0 0) (end 12.25 0) (layer Dwgs.User) (width 0.15))
-    (fp_arc (start -10.15 -7.25) (end -10.15 -9.8) (angle -90) (layer B.Fab) (width 0.1))
-    (fp_arc (start 10.15 -7.25) (end 10.15 -9.8) (angle 90) (layer B.Fab) (width 0.1))
-    (fp_line (start -12.85 -1.9) (end -12.85 -7.3) (layer B.SilkS) (width 0.12))
-    (fp_line (start 12.85 -1.9) (end 12.85 -7.3) (layer B.SilkS) (width 0.12))
-    (fp_arc (start 10.15 -7.25) (end 10.15 -9.95) (angle 90) (layer B.SilkS) (width 0.12))
-    (fp_arc (start -10.15 -7.25) (end -10.15 -9.95) (angle -90) (layer B.SilkS) (width 0.12))
-    (fp_arc (start 0 -21) (end -9.6 -9.58) (angle -80) (layer B.Fab) (width 0.1))
-    (fp_arc (start -10.15 -9) (end -10.15 -9.8) (angle 45) (layer B.Fab) (width 0.1))
-    (fp_arc (start 10.15 -9) (end 10.15 -9.8) (angle -45) (layer B.Fab) (width 0.1))
-    (fp_arc (start -10.15 -9) (end -10.15 -9.95) (angle 45) (layer B.SilkS) (width 0.12))
-    (fp_arc (start 10.15 -9) (end 10.15 -9.95) (angle -45) (layer B.SilkS) (width 0.12))
-    (fp_arc (start 0 -21) (end -9.55 -9.73) (angle -80) (layer B.SilkS) (width 0.12))
-    (fp_arc (start -12.7 0) (end -13.35 -1.95) (angle -143) (layer B.CrtYd) (width 0.05))
-    (fp_arc (start 12.7 0) (end 13.35 -1.95) (angle 143) (layer B.CrtYd) (width 0.05))
-    (fp_arc (start -10.15 -7.25) (end -10.15 -10.45) (angle -90) (layer B.CrtYd) (width 0.05))
-    (fp_arc (start 10.15 -7.25) (end 10.15 -10.45) (angle 90) (layer B.CrtYd) (width 0.05))
-    (fp_arc (start -10.15 -9) (end -10.15 -10.45) (angle 45) (layer B.CrtYd) (width 0.05))
-    (fp_arc (start 10.15 -9) (end 10.15 -10.45) (angle -45) (layer B.CrtYd) (width 0.05))
-    (fp_arc (start 0 -21) (end -9.15 -10.05) (angle -3.2) (layer B.CrtYd) (width 0.05))
-    (fp_arc (start 0 0) (end 0 -12.8) (angle -41.7) (layer B.CrtYd) (width 0.05))
-    (fp_arc (start 0 -21) (end 9.15 -10.05) (angle 3.2) (layer B.CrtYd) (width 0.05))
-    (fp_arc (start 0 0) (end 0 -12.8) (angle 41.7) (layer B.CrtYd) (width 0.05))
-    (fp_text user %R (at 0 0 90) (layer B.Fab)
-      (effects (font (size 1 1) (thickness 0.15)) (justify mirror))
-    )
-    (pad 2 smd rect (at 0 0 270) (size 8 8) (layers B.Cu B.Mask)
-      (net 1 GND))
-    (pad 1 thru_hole circle (at 12.7 0 270) (size 3 3) (drill 1.9) (layers *.Cu *.Mask)
-      (net 2 +3V0))
-    (pad 1 thru_hole circle (at -12.7 0 270) (size 3 3) (drill 1.9) (layers *.Cu *.Mask)
-      (net 2 +3V0))
-    (model ${KISYS3DMOD}/Battery.3dshapes/BatteryHolder_Keystone_3009_1x2450.wrl
-      (at (xyz 0 0 0))
-      (scale (xyz 1 1 1))
