File: pcb/snowman_pcb.sch (KiCad schematic (older format))
At the start: 7 parts, among them SW1 SW_SPDT

Commit message: Pcb - all components in place
Parts:
- D5: footprint snowman_pcb:LED_1206_3216Metric_ReverseMount_NoHole1.8x2.4mm -> snowman_pcb:LED_D3.0mm_Horizontal_O1.27mm_Z2.0mm
Changed lines of the file:
@@
 LIBS:power
 LIBS:74xx
+LIBS:snowman_pcb-cache
 EELAYER 30 0
 EELAYER END
@@
 F 0 "D5" V 4839 1733 50  0000 R CNN
 F 1 "LED" V 4748 1733 50  0000 R CNN
-F 2 "snowman_pcb:LED_1206_3216Metric_ReverseMount_NoHole1.8x2.4mm" H 4800 1850 50  0001 C CNN
+F 2 "snowman_pcb:LED_D3.0mm_Horizontal_O1.27mm_Z2.0mm" H 4800 1850 50  0001 C CNN
 F 3 "~" H 4800 1850 50  0001 C CNN
 	1    4800 1850

Commit message: Finished revision 1
Connections:
- no-connect marks 0 -> 1
Changed lines of the file:
@@
 	2600 1650 2600 1600
-Wire Wire Line
-	3000 1700 3300 1700
-Connection ~ 3300 1700
 Wire Wire Line
 	3300 1700 3750 1700
@@
 Wire Wire Line
 	4500 2000 4800 2000
+Wire Wire Line
+	3300 1700 3000 1700
+Connection ~ 3300 1700
+NoConn ~ 3000 1500
 $EndSCHEMATC

Commit message: Remove invalid footprint, add readme and licence
Parts:
- BT1: footprint snowman_pcb:BatteryHolder_THT_CR2032 -> Battery:BatteryHolder_Keystone_3009_1x2450
Changed lines of the file:
@@
 F 0 "BT1" H 1868 1946 50  0000 L CNN
 F 1 "Battery_Cell" H 1868 1855 50  0000 L CNN
-F 2 "snowman_pcb:BatteryHolder_THT_CR2032" V 1750 1910 50  0001 C CNN
+F 2 "Battery:BatteryHolder_Keystone_3009_1x2450" V 1750 1910 50  0001 C CNN
 F 3 "~" V 1750 1910 50  0001 C CNN
 	1    1750 1850
